Commit message: Update arguments for alice and bob

File: my_dual_robot_cell/my_dual_robot_cell_control/urdf/my_dual_robot_cell_controlled.urdf.xacro (robot description, xacro)
@@ -2,36 +2,38 @@
 <robot name="my_dual_robot_cell" xmlns:xacro="http://ros.org/wiki/xacro">
   <!--First, include the macro from our custom description-->
-  <xacro:include filename="$(find my_dual_robot_cell_description)/urdf/my_dual_robot_cell_macro.xacro"/>
+  <xacro:include
+    filename="$(find my_dual_robot_cell_description)/urdf/my_dual_robot_cell_macro.xacro" />
   <!--The driver already provides a control tag for the UR arm, we can directly include-->
-  <xacro:include filename="$(find ur_robot_driver)/urdf/ur.ros2_control.xacro"/>
+  <xacro:include filename="$(find ur_robot_driver)/urdf/ur.ros2_control.xacro" />
   <!--We need to specify the arguments used for parametrizing our description-->
-  <xacro:arg name="alice_ur_type" default="ur3"/>
-  <xacro:arg name="alice_joint_limits_parameters_file" default="$(find ur_description)/config/$(arg alice_ur_type)/joint_limits.yaml"/>
-  <xacro:arg name="alice_kinematics_parameters_file" default="$(find ur_description)/config/$(arg alice_ur_type)/default_kinematics.yaml"/>
-  <xacro:arg name="alice_physical_parameters_file" default="$(find ur_description)/config/$(arg alice_ur_type)/physical_parameters.yaml"/>
-  <xacro:arg name="alice_visual_parameters_file" default="$(find ur_description)/config/$(arg alice_ur_type)/visual_parameters.yaml"/>
-  <xacro:arg name="bob_ur_type" default="ur3"/>
-  <xacro:arg name="bob_joint_limits_parameters_file" default="$(find ur_description)/config/$(arg bob_ur_type)/joint_limits.yaml"/>
-  <xacro:arg name="bob_kinematics_parameters_file" default="$(find ur_description)/config/$(arg bob_ur_type)/default_kinematics.yaml"/>
-  <xacro:arg name="bob_physical_parameters_file" default="$(find ur_description)/config/$(arg bob_ur_type)/physical_parameters.yaml"/>
-  <xacro:arg name="bob_visual_parameters_file" default="$(find ur_description)/config/$(arg bob_ur_type)/visual_parameters.yaml"/>
+  <xacro:arg name="alice_ur_type" default="ur3" />
+  <xacro:arg name="alice_joint_limits_parameters_file" default="$(find ur_description)/config/$(arg alice_ur_type)/joint_limits.yaml" />
+  <xacro:arg name="alice_kinematics_parameters_file" default="$(find ur_description)/config/$(arg alice_ur_type)/default_kinematics.yaml" />
+  <xacro:arg name="alice_physical_parameters_file" default="$(find ur_description)/config/$(arg alice_ur_type)/physical_parameters.yaml" />
+  <xacro:arg name="alice_visual_parameters_file" default="$(find ur_description)/config/$(arg alice_ur_type)/visual_parameters.yaml" />
+  <xacro:arg name="bob_ur_type" default="ur3" />
+  <xacro:arg name="bob_joint_limits_parameters_file" default="$(find ur_description)/config/$(arg bob_ur_type)/joint_limits.yaml" />
+  <xacro:arg name="bob_kinematics_parameters_file" default="$(find ur_description)/config/$(arg bob_ur_type)/default_kinematics.yaml" />
+  <xacro:arg name="bob_physical_parameters_file" default="$(find ur_description)/config/$(arg bob_ur_type)/physical_parameters.yaml" />
+  <xacro:arg name="bob_visual_parameters_file" default="$(find ur_description)/config/$(arg bob_ur_type)/visual_parameters.yaml" />
+  <xacro:arg name="alice_use_mock_hardware" default="false" />
+  <xacro:arg name="alice_mock_sensor_commands" default="false" />
+  <xacro:arg name="alice_robot_ip" default="192.168.0.101" />
+  <xacro:arg name="alice_reverse_port" default="50006" />
+  <xacro:arg name="alice_script_sender_port" default="50007" />
+  <xacro:arg name="alice_script_command_port" default="50010" />
+  <xacro:arg name="alice_trajectory_port" default="50009" />
+  <xacro:arg name="bob_use_mock_hardware" default="false" />
+  <xacro:arg name="bob_mock_sensor_commands" default="false" />
+  <xacro:arg name="bob_robot_ip" default="192.168.0.100" />
+  <xacro:arg name="bob_reverse_port" default="50001" />
+  <xacro:arg name="bob_script_sender_port" default="50002" />
+  <xacro:arg name="bob_script_command_port" default="50004" />
+  <xacro:arg name="bob_trajectory_port" default="50003" />
   <xacro:arg name="headless_mode" default="false" />
-  <xacro:arg name="ur_script_filename" default="$(find ur_client_library)/resources/external_control.urscript"/>
-  <xacro:arg name="ur_output_recipe_filename" default="$(find ur_robot_driver)/resources/rtde_output_recipe.txt"/>
-  <xacro:arg name="ur_input_recipe_filename" default="$(find ur_robot_driver)/resources/rtde_input_recipe.txt"/>
-  <xacro:arg name="use_mock_hardware" default="true" />
-  <xacro:arg name="mock_sensor_commands" default="false" />
-  <xacro:arg name="alice_robot_ip" default="192.168.0.101"/>
-  <xacro:arg name="alice_reverse_port" default="50001"/>
-  <xacro:arg name="alice_script_sender_port" default="50002"/>
-  <xacro:arg name="alice_script_command_port" default="50004"/>
-  <xacro:arg name="alice_trajectory_port" default="50003"/>
-  <xacro:arg name="bob_robot_ip" default="192.168.0.100"/>
-  <xacro:arg name="bob_reverse_port" default="50006"/>
-  <xacro:arg name="bob_script_sender_port" default="50007"/>
-  <xacro:arg name="bob_script_command_port" default="50010"/>
-  <xacro:arg name="bob_trajectory_port" default="50009"/>
+  <xacro:arg name="ur_script_filename" default="$(find ur_client_library)/resources/external_control.urscript" />
+  <xacro:arg name="ur_output_recipe_filename" default="$(find ur_robot_driver)/resources/rtde_output_recipe.txt" />
+  <xacro:arg name="ur_input_recipe_filename" default="$(find ur_robot_driver)/resources/rtde_input_recipe.txt" />
   <link name="world" />
-  <!--Create the scene description including the robot-->
   <xacro:my_dual_robot_cell
     parent="world"
@@ -46,8 +48,7 @@
     bob_physical_parameters_file="$(arg bob_physical_parameters_file)"
     bob_visual_parameters_file="$(arg bob_visual_parameters_file)"
-    >
-      <origin xyz="0 0 1" rpy="0 0 0" />
+  >
+    <origin xyz="0 0 1" rpy="0 0 0" />
   </xacro:my_dual_robot_cell>
-  <!--Create the control tag for the UR robot-->
   <xacro:ur_ros2_control
     name="alice"
@@ -58,6 +59,6 @@
     output_recipe_filename="$(arg ur_output_recipe_filename)"
     input_recipe_filename="$(arg ur_input_recipe_filename)"
-    use_mock_hardware="$(arg use_mock_hardware)"
-    mock_sensor_commands="$(arg mock_sensor_commands)"
+    use_mock_hardware="$(arg alice_use_mock_hardware)"
+    alice_mock_sensor_commands="$(arg alice_mock_sensor_commands)"
     headless_mode="$(arg headless_mode)"
     reverse_port="$(arg alice_reverse_port)"
@@ -74,6 +75,6 @@
     output_recipe_filename="$(arg ur_output_recipe_filename)"
     input_recipe_filename="$(arg ur_input_recipe_filename)"
-    use_mock_hardware="$(arg use_mock_hardware)"
-    mock_sensor_commands="$(arg mock_sensor_commands)"
+    use_mock_hardware="$(arg bob_use_mock_hardware)"
+    bob_mock_sensor_commands="$(arg bob_mock_sensor_commands)"
     headless_mode="$(arg headless_mode)"
     reverse_port="$(arg bob_reverse_port)"
@@ -82,4 +83,3 @@
     trajectory_port="$(arg bob_trajectory_port)"
   />
-  <!--If you had more controlled devices in your description, e.g. a gripper, you can add another ros2_control tag here-->
 </robot>
