Commit message: kinematics_hash now automatically read from kinematics_params

File: my_robot_cell/my_robot_cell_control/urdf/my_robot_cell_controlled.urdf.xacro (robot description, xacro)
@@ -20,6 +20,7 @@
   <xacro:arg name="use_fake_hardware" default="false" />
   <xacro:arg name="fake_sensor_commands" default="false" />
-  <!--find hash_kinematics in calibration yaml-->
-  <xacro:arg name="hash_kinematics" default="calib_4890363623803256388" />
+  <!--find hash_kinematics in kinematics_params-->
+  <xacro:property name="kinematics_params_file" value="$(arg kinematics_params)"/>
+  <xacro:property name="kinematics_hash" value="${xacro.load_yaml(kinematics_params_file)['kinematics']['hash']}"/>
   <link name="world" />
   <!--Create the scene description including the robot-->
@@ -38,5 +39,5 @@
     name="$(arg ur_type)"
     tf_prefix="$(arg ur_type)_"
-    hash_kinematics="$(arg hash_kinematics)"
+    hash_kinematics="${kinematics_hash}"
     robot_ip="$(arg robot_ip)"
     script_filename="$(arg ur_script_filename)"

Commit message: Update Humble documentation to match the Humble state (#11)
As the Humble description is structured differently to the Jazzy+ description, the example has to be restructured, as well.

---------

Co-authored-by: Felix Exner <feex@universal-robots.com>

File: my_robot_cell/my_robot_cell_control/urdf/my_robot_cell_controlled.urdf.xacro (robot description, xacro)
@@ -3,12 +3,14 @@
   <!--First, include the macro from our custom description-->
   <xacro:include filename="$(find my_robot_cell_description)/urdf/my_robot_cell_macro.xacro"/>
-  <!--The driver already provides a control tag for the UR arm, we can directly include-->
-  <xacro:include filename="$(find ur_robot_driver)/urdf/ur.ros2_control.xacro"/>
+  <!--The ur_description package already provides a control tag for the UR arm, we can directly include-->
+  <xacro:include filename="$(find ur_description)/urdf/ur.ros2_control.xacro"/>
   <!--We need to specify the arguments used for parametrizing our description-->
+  <!--Create a folder for wanted ur_type and copy those files from ur_description package in there; copied only ur20 files -->
+  <!--You could as well point to ur_description but this way you make sure you use the same files as start_robot.launch.py which searches in runtime_config_package for joint_limits.yaml, physical_parameters.yaml, visual_parameters.yaml and in description_package for default_kinematics.yaml (last one can be overwritten)-->
   <xacro:arg name="ur_type" default="ur20"/>
-  <xacro:arg name="joint_limit_parameters_file" default="$(find ur_description)/config/$(arg ur_type)/joint_limits.yaml"/>
-  <xacro:arg name="kinematics_parameters_file" default="$(find ur_description)/config/$(arg ur_type)/default_kinematics.yaml"/>
-  <xacro:arg name="physical_parameters_file" default="$(find ur_description)/config/$(arg ur_type)/physical_parameters.yaml"/>
-  <xacro:arg name="visual_parameters_file" default="$(find ur_description)/config/$(arg ur_type)/visual_parameters.yaml"/>
+  <xacro:arg name="joint_limit_params" default="$(find my_robot_cell_control)/config/$(arg ur_type)/joint_limits.yaml"/>
+  <xacro:arg name="kinematics_params" default="$(find my_robot_cell_control)/config/$(arg ur_type)/default_kinematics.yaml"/>
+  <xacro:arg name="physical_params" default="$(find my_robot_cell_control)/config/$(arg ur_type)/physical_parameters.yaml"/>
+  <xacro:arg name="visual_params" default="$(find my_robot_cell_control)/config/$(arg ur_type)/visual_parameters.yaml"/>
   <xacro:arg name="robot_ip" default="0.0.0.0"/>
   <xacro:arg name="headless_mode" default="false" />
@@ -16,6 +18,9 @@
   <xacro:arg name="ur_output_recipe_filename" default="$(find ur_robot_driver)/resources/rtde_output_recipe.txt"/>
   <xacro:arg name="ur_input_recipe_filename" default="$(find ur_robot_driver)/resources/rtde_input_recipe.txt"/>
-  <xacro:arg name="use_mock_hardware" default="false" />
-  <xacro:arg name="mock_sensor_commands" default="false" />
+  <xacro:arg name="use_fake_hardware" default="false" />
+  <xacro:arg name="fake_sensor_commands" default="false" />
+  <!--find hash_kinematics in kinematics_params-->
+  <xacro:property name="kinematics_params_file" value="$(arg kinematics_params)"/>
+  <xacro:property name="kinematics_hash" value="${xacro.load_yaml(kinematics_params_file)['kinematics']['hash']}"/>
   <link name="world" />
   <!--Create the scene description including the robot-->
@@ -23,8 +28,8 @@
     parent="world"
     ur_type="$(arg ur_type)"
-    joint_limits_parameters_file="$(arg joint_limit_parameters_file)"
-    kinematics_parameters_file="$(arg kinematics_parameters_file)"
-    physical_parameters_file="$(arg physical_parameters_file)"
-    visual_parameters_file="$(arg visual_parameters_file)"
+    joint_limits_parameters_file="$(arg joint_limit_params)"
+    kinematics_parameters_file="$(arg kinematics_params)"
+    physical_parameters_file="$(arg physical_params)"
+    visual_parameters_file="$(arg visual_params)"
   >
     <origin xyz="0 0 1" rpy="0 0 0" />
@@ -34,11 +39,11 @@
     name="$(arg ur_type)"
     tf_prefix="$(arg ur_type)_"
-    kinematics_parameters_file="$(arg kinematics_parameters_file)"
+    hash_kinematics="${kinematics_hash}"
     robot_ip="$(arg robot_ip)"
     script_filename="$(arg ur_script_filename)"
     output_recipe_filename="$(arg ur_output_recipe_filename)"
     input_recipe_filename="$(arg ur_input_recipe_filename)"
-    use_mock_hardware="$(arg use_mock_hardware)"
-    mock_sensor_commands="$(arg mock_sensor_commands)"
+    use_fake_hardware="$(arg use_fake_hardware)"
+    fake_sensor_commands="$(arg fake_sensor_commands)"
     headless_mode="$(arg headless_mode)"
   />
