Commit message: Re use mesh files from custom_workcell in the my_robot_cell package

File: my_dual_robot_cell/my_dual_robot_cell_description/urdf/my_dual_robot_cell_macro.xacro (robot description, xacro)
@@ -24,5 +24,5 @@
       <visual>
         <geometry>
-          <mesh filename="package://my_dual_robot_cell_description/meshes/fzi_table.dae"/>
+          <mesh filename="package://my_robot_cell_description/meshes/fzi_table.dae"/>
         </geometry>
         <origin rpy="0 0 0" xyz="0.75 0.5 -1"/>
@@ -30,5 +30,5 @@
       <collision>
         <geometry>
-          <mesh filename="package://my_dual_robot_cell_description/meshes/fzi_table.dae"/>
+          <mesh filename="package://my_robot_cell_description/meshes/fzi_table.dae"/>
         </geometry>
         <origin rpy="0 0 0" xyz="0.75 0.5 -1"/>
@@ -38,10 +38,10 @@
       <visual>
         <geometry>
-          <mesh filename="package://my_dual_robot_cell_description/meshes/171005_Motek_Monitor_L.dae"/>
+          <mesh filename="package://my_robot_cell_description/meshes/171005_Motek_Monitor_L.dae"/>
         </geometry>
       </visual>
       <collision>
         <geometry>
-          <mesh filename="package://my_dual_robot_cell_description/meshes/171005_Motek_Monitor_L.dae"/>
+          <mesh filename="package://my_robot_cell_description/meshes/171005_Motek_Monitor_L.dae"/>
         </geometry>
       </collision>
@@ -58,5 +58,5 @@
       <visual>
         <geometry>
-          <mesh filename="package://my_dual_robot_cell_description/meshes/wall.dae"/>
+          <mesh filename="package://my_robot_cell_description/meshes/wall.dae"/>
         </geometry>
       </visual>

Commit message: Move alice and bob robots to a slightly better position

File: my_dual_robot_cell/my_dual_robot_cell_description/urdf/my_dual_robot_cell_macro.xacro (robot description, xacro)
@@ -77,5 +77,5 @@
       <parent link="table"/>
       <child link="alice_robot_mount"/>
-      <origin xyz="0.3 0.85 0" rpy="0 0 ${pi}" />
+      <origin xyz="0.5 0.3 0" rpy="0 0 ${pi}" />
     </joint>
     <link name="bob_robot_mount"/>
@@ -83,5 +83,5 @@
       <parent link="table"/>
       <child link="bob_robot_mount"/>
-      <origin xyz="1.0 0.85 0" rpy="0 0 ${pi}" />
+      <origin xyz="1.2 0.3 0" rpy="0 0 ${pi}" />
     </joint>
     <!--Creates the 1st Robot-->

Commit message: dual arm tutorial documentation

File: my_dual_robot_cell/my_dual_robot_cell_description/urdf/my_dual_robot_cell_macro.xacro (robot description, xacro)
@@ -77,5 +77,5 @@
       <parent link="table"/>
       <child link="alice_robot_mount"/>
-      <origin xyz="0.5 0.3 0" rpy="0 0 ${pi}" />
+      <origin xyz="0.2 0.3 0" rpy="0 0 ${pi}" />
     </joint>
     <link name="bob_robot_mount"/>
